File: hardware/display.kicad_sch (KiCad schematic)
At the start: 2 parts

Commit message: train schematics
Other:
- company: Erdapfel -> Frisius
Changed lines of the file:
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@@
   (title_block
     (rev "A")
-    (company "Erdapfel")
+    (company "Frisius")
   )
   (hierarchical_label "STATUS_LED" (shape input) (at 41.91 85.09 0)

Commit message: started b2b and power
Connections:
- net STATUS_LED: now also J?.3 (Pin_3)
- net GND: now reaches J?.1 (Pin_1)
- net GND: now also J?.19 (Pin_19), J?.2 (Pin_2), J?.5 (Pin_5), J?.6 (Pin_6), J?.SH (Shield)
- net USR_BTN.NAV_A: now reaches J?.10 (Pin_10)
- net DISPLAY.SCLK: now reaches J?.11 (Pin_11)
- net USR_BTN.PWR: now reaches J?.12 (Pin_12)
- net DISPLAY.CS: now reaches J?.13 (Pin_13)
- net DISPLAY.DC: now reaches J?.15 (Pin_15)
- net SENSOR_I2C.SDA: now reaches J?.16 (Pin_16)
- net DISPLAY.BL: now reaches J?.17 (Pin_17)
- net SENSOR_I2C.SCL: now reaches J?.18 (Pin_18)
- net VDD_AUX_EN: now reaches J?.4 (Pin_4)
- net DISPLAY.MOSI: now reaches J?.7 (Pin_7)
- net DISPLAY.MISO: now reaches J?.9 (Pin_9)
Other:
- moved on the sheet: J?
Changed lines of the file:
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@@
     (company "Frisius")
   )
-  (hierarchical_label "STATUS_LED" (shape input) (at 41.91 85.09 0)
+  (junction (at 93.98 97.79) (diameter 0) (color 0 0 0 0)
+  )
+  (junction (at 101.6 73.66) (diameter 0) (color 0 0 0 0)
+  )
+  (junction (at 86.36 73.66) (diameter 0) (color 0 0 0 0)
+  )
+  (junction (at 86.36 91.44) (diameter 0) (color 0 0 0 0)
+  )
+  (bus_entry (at 115.57 78.74) (size 2.54 -2.54)
+    (stroke (width 0) (type default) (color 0 0 0 0))
+  )
+  (bus_entry (at 115.57 81.28) (size 2.54 -2.54)
+    (stroke (width 0) (type default) (color 0 0 0 0))
+  )
+  (bus_entry (at 73.66 86.36) (size -2.54 -2.54)
+    (stroke (width 0) (type default) (color 0 0 0 0))
+  )
+  (bus_entry (at 73.66 88.9) (size -2.54 -2.54)
+    (stroke (width 0) (type default) (color 0 0 0 0))
+  )
+  (bus_entry (at 73.66 83.82) (size -2.54 -2.54)
+    (stroke (width 0) (type default) (color 0 0 0 0))
+  )
+  (bus_entry (at 73.66 76.2) (size -2.54 -2.54)
+    (stroke (width 0) (type default) (color 0 0 0 0))
+  )
+  (bus_entry (at 115.57 88.9) (size 2.54 -2.54)
+    (stroke (width 0) (type default) (color 0 0 0 0))
+  )
+  (bus_entry (at 73.66 81.28) (size -2.54 -2.54)
+    (stroke (width 0) (type default) (color 0 0 0 0))
+  )
+  (bus_entry (at 115.57 86.36) (size 2.54 -2.54)
+    (stroke (width 0) (type default) (color 0 0 0 0))
+  )
+  (bus_entry (at 73.66 78.74) (size -2.54 -2.54)
+    (stroke (width 0) (type default) (color 0 0 0 0))
+  )
+  (bus (pts (xy 69.85 72.39) (xy 71.12 73.66))
+    (stroke (width 0) (type default) (color 0 0 0 0))
+  )
+  (wire (pts (xy 73.66 86.36) (xy 87.63 86.36))
+    (stroke (width 0) (type default) (color 0 0 0 0))
+  )
+  (wire (pts (xy 87.63 71.12) (xy 76.2 71.12))
+    (stroke (width 0) (type default) (color 0 0 0 0))
+  )
+  (bus (pts (xy 71.12 76.2) (xy 71.12 73.66))
+    (stroke (width 0) (type default) (color 0 0 0 0))
+  )
+  (wire (pts (xy 100.33 68.58) (xy 101.6 68.58))
+    (stroke (width 0) (type default) (color 0 0 0 0))
+  )
+  (wire (pts (xy 101.6 97.79) (xy 93.98 97.79))
+    (stroke (width 0) (type default) (color 0 0 0 0))
+  )
+  (wire (pts (xy 100.33 78.74) (xy 115.57 78.74))
+    (stroke (width 0) (type default) (color 0 0 0 0))
+  )
+  (wire (pts (xy 86.36 68.58) (xy 86.36 73.66))
+    (stroke (width 0) (type default) (color 0 0 0 0))
+  )
+  (wire (pts (xy 76.2 71.12) (xy 72.39 67.31))
+    (stroke (width 0) (type default) (color 0 0 0 0))
+  )
+  (wire (pts (xy 100.33 86.36) (xy 115.57 86.36))
+    (stroke (width 0) (type default) (color 0 0 0 0))
+  )
+  (wire (pts (xy 73.66 83.82) (xy 87.63 83.82))
+    (stroke (width 0) (type default) (color 0 0 0 0))
+  )
+  (bus (pts (xy 71.12 78.74) (xy 71.12 76.2))
+    (stroke (width 0) (type default) (color 0 0 0 0))
+  )
+  (wire (pts (xy 86.36 73.66) (xy 86.36 91.44))
+    (stroke (width 0) (type default) (color 0 0 0 0))
+  )
+  (wire (pts (xy 73.66 76.2) (xy 87.63 76.2))
+    (stroke (width 0) (type default) (color 0 0 0 0))
+  )
+  (wire (pts (xy 113.03 71.12) (xy 100.33 71.12))
+    (stroke (width 0) (type default) (color 0 0 0 0))
+  )
+  (bus (pts (xy 67.31 72.39) (xy 69.85 72.39))
+    (stroke (width 0) (type default) (color 0 0 0 0))
+  )
+  (bus (pts (xy 121.92 74.93) (xy 119.38 74.93))
+    (stroke (width 0) (type default) (color 0 0 0 0))
+  )
+  (wire (pts (xy 86.36 97.79) (xy 93.98 97.79))
+    (stroke (width 0) (type default) (color 0 0 0 0))
+  )
+  (bus (pts (xy 118.11 83.82) (xy 119.38 82.55))
+    (stroke (width 0) (type default) (color 0 0 0 0))
+  )
+  (wire (pts (xy 113.03 71.12) (xy 116.84 67.31))
+    (stroke (width 0) (type default) (color 0 0 0 0))
+  )
+  (wire (pts (xy 100.33 81.28) (xy 115.57 81.28))
+    (stroke (width 0) (type default) (color 0 0 0 0))
+  )
+  (wire (pts (xy 116.84 67.31) (xy 119.38 67.31))
+    (stroke (width 0) (type default) (color 0 0 0 0))
+  )
+  (wire (pts (xy 101.6 73.66) (xy 101.6 97.79))
+    (stroke (width 0) (type default) (color 0 0 0 0))
+  )
+  (wire (pts (xy 73.66 81.28) (xy 87.63 81.28))
+    (stroke (width 0) (type default) (color 0 0 0 0))
+  )
+  (bus (pts (xy 71.12 81.28) (xy 71.12 78.74))
+    (stroke (width 0) (type default) (color 0 0 0 0))
+  )
+  (bus (pts (xy 119.38 82.55) (xy 121.92 82.55))
+    (stroke (width 0) (type default) (color 0 0 0 0))
+  )
+  (bus (pts (xy 71.12 86.36) (xy 71.12 83.82))
+    (stroke (width 0) (type default) (color 0 0 0 0))
+  )
+  (wire (pts (xy 72.39 67.31) (xy 69.85 67.31))
+    (stroke (width 0) (type default) (color 0 0 0 0))
+  )
+  (wire (pts (xy 87.63 91.44) (xy 86.36 91.44))
+    (stroke (width 0) (type default) (color 0 0 0 0))
+  )
+  (wire (pts (xy 73.66 78.74) (xy 87.63 78.74))
+    (stroke (width 0) (type default) (color 0 0 0 0))
+  )
+  (wire (pts (xy 86.36 91.44) (xy 86.36 97.79))
+    (stroke (width 0) (type default) (color 0 0 0 0))
+  )
+  (bus (pts (xy 71.12 83.82) (xy 71.12 81.28))
+    (stroke (width 0) (type default) (color 0 0 0 0))
+  )
+  (bus (pts (xy 118.11 86.36) (xy 118.11 83.82))
+    (stroke (width 0) (type default) (color 0 0 0 0))
+  )
+  (wire (pts (xy 93.98 99.06) (xy 93.98 97.79))
+    (stroke (width 0) (type default) (color 0 0 0 0))
+  )
+  (wire (pts (xy 93.98 97.79) (xy 93.98 96.52))
+    (stroke (width 0) (type default) (color 0 0 0 0))
+  )
+  (wire (pts (xy 73.66 88.9) (xy 87.63 88.9))
+    (stroke (width 0) (type default) (color 0 0 0 0))
+  )
+  (bus (pts (xy 118.11 76.2) (xy 118.11 78.74))
+    (stroke (width 0) (type default) (color 0 0 0 0))
+  )
+  (wire (pts (xy 101.6 73.66) (xy 100.33 73.66))
+    (stroke (width 0) (type default) (color 0 0 0 0))
+  )
+  (bus (pts (xy 119.38 74.93) (xy 118.11 76.2))
+    (stroke (width 0) (type default) (color 0 0 0 0))
+  )
+  (wire (pts (xy 87.63 68.58) (xy 86.36 68.58))
+    (stroke (width 0) (type default) (color 0 0 0 0))
+  )
+  (wire (pts (xy 87.63 73.66) (xy 86.36 73.66))
+    (stroke (width 0) (type default) (color 0 0 0 0))
+  )
+  (wire (pts (xy 100.33 88.9) (xy 115.57 88.9))
+    (stroke (width 0) (type default) (color 0 0 0 0))
+  )
+  (wire (pts (xy 101.6 68.58) (xy 101.6 73.66))
+    (stroke (width 0) (type default) (color 0 0 0 0))
+  )
+  (label "DISPLAY.DC" (at 74.93 86.36 0)
+    (effects (font (size 0.8 0.8)) (justify left bottom))
+  )
+  (label "USR_BTN.NAV_A" (at 114.3 78.74 180)
+    (effects (font (size 0.8 0.8)) (justify right bottom))
+  )
+  (label "SENSOR_I2C.SDA" (at 114.3 86.36 180)
+    (effects (font (size 0.8 0.8)) (justify right bottom))
+  )
+  (label "DISPLAY.MOSI" (at 74.93 76.2 0)
+    (effects (font (size 0.8 0.8)) (justify left bottom))
+  )
+  (label "DISPLAY.CS" (at 74.93 83.82 0)
+    (effects (font (size 0.8 0.8)) (justify left bottom))
+  )
+  (label "DISPLAY.BL" (at 74.93 88.9 0)
+    (effects (font (size 0.8 0.8)) (justify left bottom))
+  )
+  (label "SENSOR_I2C.SCL" (at 114.3 88.9 180)
+    (effects (font (size 0.8 0.8)) (justify right bottom))
+  )
+  (label "DISPLAY.SCLK" (at 74.93 81.28 0)
+    (effects (font (size 0.8 0.8)) (justify left bottom))
+  )
+  (label "DISPLAY.MISO" (at 74.93 78.74 0)
+    (effects (font (size 0.8 0.8)) (justify left bottom))
+  )
+  (label "USR_BTN.PWR" (at 114.3 81.28 180)
+    (effects (font (size 0.8 0.8)) (justify right bottom))
+  )
+  (hierarchical_label "USR_BTN{NAV_A PWR}" (shape input) (at 121.92 74.93 0)
     (effects (font (size 0.8 0.8)) (justify left))
   )
-  (hierarchical_label "DISPLAY{MOSI MISO SCLK CS DC BL}" (shape bidirectional) (at 41.91 72.39 0)
+  (hierarchical_label "VDD_AUX_EN" (shape input) (at 119.38 67.31 0)
     (effects (font (size 0.8 0.8)) (justify left))
   )
-  (hierarchical_label "BTN{PWR NAV_A}" (shape output) (at 41.91 82.55 0)
+  (hierarchical_label "SENSOR_I2C{SDA SCL}" (shape bidirectional) (at 121.92 82.55 0)
     (effects (font (size 0.8 0.8)) (justify left))
   )
-  (hierarchical_label "SENSOR_I2C{SDA SCL}" (shape bidirectional) (at 41.91 74.93 0)
-    (effects (font (size 0.8 0.8)) (justify left))
-  )
-  (symbol (lib_id "Connector_Generic_Shielded:Conn_02x10_Odd_Even_Shielded") (at 71.12 45.72 0) (unit 1)
+  (hierarchical_label "STATUS_LED" (shape output) (at 69.85 67.31 180)
+    (effects (font (size 0.8 0.8)) (justify right))
+  )
+  (hierarchical_label "DISPLAY{MOSI MISO SCLK CS DC BL}" (shape bidirectional) (at 67.31 72.39 180)
+    (effects (font (size 0.8 0.8)) (justify right))
+  )
+  (symbol (lib_id "Connector_Generic_Shielded:Conn_02x10_Odd_Even_Shielded") (at 92.71 78.74 0) (unit 1)
     (in_bom yes) (on_board yes) (fields_autoplaced)
-    (property "Reference" "J?" (id 0) (at 72.39 29.21 0)
+    (property "Reference" "J?" (id 0) (at 93.98 62.23 0)
       (effects (font (size 0.8 0.8)))
     )
-    (property "Value" "Conn_02x10_Odd_Even_Shielded" (id 1) (at 72.39 31.75 0)
+    (property "Value" "Conn_02x10_Odd_Even_Shielded" (id 1) (at 93.98 64.77 0)
       (effects (font (size 0.8 0.8)))
     )
-    (property "Footprint" "" (id 2) (at 71.12 45.72 0)
-      (effects (font (size 0.8 0.8)) hide)
-    )
-    (property "Datasheet" "~" (id 3) (at 71.12 45.72 0)
+    (property "Footprint" "" (id 2) (at 92.71 78.74 0)
+      (effects (font (size 0.8 0.8)) hide)
+    )
+    (property "Datasheet" "~" (id 3) (at 92.71 78.74 0)
       (effects (font (size 0.8 0.8)) hide)
     )
@@
     (pin "SH")
   )
+  (symbol (lib_id "power:GND") (at 93.98 99.06 0) (unit 1)
+    (in_bom yes) (on_board yes) (fields_autoplaced)
+    (property "Reference" "#PWR?" (id 0) (at 93.98 105.41 0)
+      (effects (font (size 0.8 0.8)) hide)
+    )
+    (property "Value" "GND" (id 1) (at 93.98 104.14 0)
+      (effects (font (size 0.8 0.8)) hide)
+    )
+    (property "Footprint" "" (id 2) (at 93.98 99.06 0)
+      (effects (font (size 0.8 0.8)) hide)
+    )
+    (property "Datasheet" "" (id 3) (at 93.98 99.06 0)
+      (effects (font (size 0.8 0.8)) hide)
+    )
+    (pin "1")
+  )
   (symbol (lib_id "Connector_Generic_Shielded:Conn_02x10_Odd_Even_Shielded") (at 137.16 45.72 0) (unit 1)

Commit message: ready for first review
Parts:
- added C? (x4): 4.7u, Capacitor_SMD:C_0805_2012Metric, symbol Device:C_Small
Connections:
- net GND: now also J?.1 (Pin_1), J?.10 (Pin_10), J?.11 (Pin_11), J?.12 (Pin_12), J?.17 (Pin_17), J?.18 (Pin_18), J?.19 (Pin_19), J?.2 (Pin_2), J?.20 (Pin_20), J?.20 (Pin_20), J?.3 (Pin_3), J?.4 (Pin_4), J?.9 (Pin_9), J?.SH (Shield), C?.2, C?.2, C?.2, C?.2
- net VCC_BKUP_3V3: now reaches J?.13 (Pin_13)
- net VCC_BKUP_3V3: now also J?.15 (Pin_15), J?.5 (Pin_5), J?.7 (Pin_7), C?.1, C?.1
- net VDD_NVDC: now reaches J?.14 (Pin_14)
- net VDD_NVDC: now also J?.16 (Pin_16), J?.6 (Pin_6), J?.8 (Pin_8), C?.1, C?.1
Other:
- note added: "Data"
- note added: "Power"
- moved on the sheet: J?

Commit message: checking footprint assignment, added current sense pac1934 for dev
Parts:
- J3, J4: renamed from J?; footprint (none) -> Connector_Molex:Molex_SlimStack_55560-0201_2x10_P0.50mm_Vertical
- gave numbers to parts that had none: 4
Changed lines of the file:
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@@
   (symbol (lib_id "power:GND") (at 193.04 116.205 0) (unit 1)
     (in_bom yes) (on_board yes) (fields_autoplaced)
-    (property "Reference" "#PWR?" (id 0) (at 193.04 122.555 0)
+    (property "Reference" "#PWR079" (id 0) (at 193.04 122.555 0)
       (effects (font (size 0.8 0.8)) hide)
     )
@@
   (symbol (lib_id "bt_power:VDD_NVDC") (at 205.74 88.265 0) (unit 1)
     (in_bom no) (on_board no)
-    (property "Reference" "U?" (id 0) (at 206.2734 88.265 0)
+    (property "Reference" "#U045" (id 0) (at 206.2734 88.265 0)
       (effects (font (size 1.27 1.27)) hide)
     )
@@
   (symbol (lib_id "Device:C_Small") (at 205.74 109.22 0) (unit 1)
     (in_bom yes) (on_board yes)
-    (property "Reference" "C?" (id 0) (at 208.28 107.95 0)
+    (property "Reference" "C75" (id 0) (at 208.28 107.95 0)
       (effects (font (size 0.8 0.8)) (justify left))
     )
@@
   (symbol (lib_id "Connector_Generic_Shielded:Conn_02x10_Odd_Even_Shielded") (at 106.68 95.885 0) (unit 1)
     (in_bom yes) (on_board yes) (fields_autoplaced)
-    (property "Reference" "J?" (id 0) (at 107.95 79.375 0)
+    (property "Reference" "J3" (id 0) (at 107.95 79.375 0)
       (effects (font (size 0.8 0.8)))
     )
@@
       (effects (font (size 0.8 0.8)))
     )
-    (property "Footprint" "" (id 2) (at 106.68 95.885 0)
+    (property "Footprint" "Connector_Molex:Molex_SlimStack_55560-0201_2x10_P0.50mm_Vertical" (id 2) (at 106.68 95.885 0)
       (effects (font (size 0.8 0.8)) hide)
     )
@@
   (symbol (lib_id "Device:C_Small") (at 180.34 109.22 0) (mirror y) (unit 1)
     (in_bom yes) (on_board yes)
-    (property "Reference" "C?" (id 0) (at 177.8 107.95 0)
+    (property "Reference" "C74" (id 0) (at 177.8 107.95 0)
       (effects (font (size 0.8 0.8)) (justify left))
     )
@@
   (symbol (lib_id "bt_power:VDD_BKUP_3V3") (at 180.34 88.265 0) (unit 1)
     (in_bom yes) (on_board yes) (fields_autoplaced)
-    (property "Reference" "#PWR?" (id 0) (at 180.34 92.075 0)
+    (property "Reference" "#PWR078" (id 0) (at 180.34 92.075 0)
       (effects (font (size 1.27 1.27)) hide)
     )
@@
   (symbol (lib_id "Device:C_Small") (at 213.36 109.22 0) (unit 1)
     (in_bom yes) (on_board yes)
-    (property "Reference" "C?" (id 0) (at 215.9 107.95 0)
+    (property "Reference" "C76" (id 0) (at 215.9 107.95 0)
       (effects (font (size 0.8 0.8)) (justify left))
     )
@@
   (symbol (lib_id "power:GND") (at 107.95 116.205 0) (unit 1)
     (in_bom yes) (on_board yes) (fields_autoplaced)
-    (property "Reference" "#PWR?" (id 0) (at 107.95 122.555 0)
+    (property "Reference" "#PWR077" (id 0) (at 107.95 122.555 0)
       (effects (font (size 0.8 0.8)) hide)
     )
@@
   (symbol (lib_id "Connector_Generic_Shielded:Conn_02x10_Odd_Even_Shielded") (at 191.77 95.885 0) (unit 1)
     (in_bom yes) (on_board yes) (fields_autoplaced)
-    (property "Reference" "J?" (id 0) (at 193.04 79.375 0)
+    (property "Reference" "J4" (id 0) (at 193.04 79.375 0)
       (effects (font (size 0.8 0.8)))
     )
@@
       (effects (font (size 0.8 0.8)))
     )
-    (property "Footprint" "" (id 2) (at 191.77 95.885 0)
+    (property "Footprint" "Connector_Molex:Molex_SlimStack_55560-0201_2x10_P0.50mm_Vertical" (id 2) (at 191.77 95.885 0)
       (effects (font (size 0.8 0.8)) hide)
     )
@@
   (symbol (lib_id "Device:C_Small") (at 172.72 109.22 0) (mirror y) (unit 1)
     (in_bom yes) (on_board yes)
-    (property "Reference" "C?" (id 0) (at 170.18 107.95 0)
-      (effects (font (size 0.8 0.8)) (justify left))
-    )
+    (property "Reference" "C73" (id 0) (at 170.18 107.95 0)
+      (effects (font (size 0.8 0.8)) (justify left))
+    )

Commit message: hardware update
Parts:
- removed C74, C75, C76: 4.7u, Capacitor_SMD:C_0805_2012Metric, symbol Device:C_Small
- added C32, C33, C34: 4.7u, Capacitor_SMD:C_0603_1608Metric, symbol Device:C_Small
- C31: renamed from C73; footprint Capacitor_SMD:C_0805_2012Metric -> Capacitor_SMD:C_0603_1608Metric
- renumbered J3 to J1, J4 to J2
Connections:
- net GND: now also J1.12 (Pin_12), J1.14 (Pin_14), C32.2, C33.2, C34.2; no longer J2.10 (Pin_10), J2.12 (Pin_12)
- net USR_BTN.NAV_A: now also J1.8 (Pin_8); no longer J1.10 (Pin_10)
- net USR_BTN.PWR: now also J1.10 (Pin_10); no longer J1.12 (Pin_12)
- net VCC_BKUP_3V3: no longer J2.13 (Pin_13), J2.15 (Pin_15)
- net VDD_NVDC: now also J2.10 (Pin_10), J2.12 (Pin_12), C33.1, C34.1
- net VDD_AUX_EN renamed VDD_CORE_EN
- new net VDD_AUX_3V3: C32.1, J2.13 (Pin_13), J2.15 (Pin_15)
Other:
- moved on the sheet: C31, J1, J2

Commit message: fixing submodule
Parts:
- removed J1, J2: Conn_02x10_Odd_Even_Shielded, Connector_Molex:Molex_SlimStack_55560-0201_2x10_P0.50mm_Vertical, symbol Connector_Generic_Shielded:Conn_02x10_Odd_Even_Shielded
- added J1: Conn_02x20_Odd_Even_Shielded, Connector_Molex:Molex_SlimStack_502426-4010_2x20_P0.40mm_Vertical, symbol Connector_Generic:Conn_02x20_Odd_Even
- C31, C32, C33, C34: value 4.7u -> 1u; Voltage 25V -> 15V
Connections:
- net VDD_AUX_3V3 is gone; now on net VCC_BKUP_3V3: C32.1
- net DISPLAY.BL: now also J1.31 (Pin_31)
- net DISPLAY.CS: now also J1.25 (Pin_25)
- net DISPLAY.DC: now also J1.27 (Pin_27)
- net DISPLAY.MISO: now also J1.21 (Pin_21)
- net DISPLAY.MOSI: now also J1.19 (Pin_19)
- net DISPLAY.SCLK: now also J1.23 (Pin_23)
- net SENSOR_I2C.SCL: now also J1.32 (Pin_32)
- net SENSOR_I2C.SDA: now also J1.30 (Pin_30)
- net USR_BTN.NAV_A: now also J1.24 (Pin_24)
- net USR_BTN.PWR: now also J1.26 (Pin_26)
- net VCC_BKUP_3V3: now also C34.1, J1.35 (Pin_35), J1.36 (Pin_36), J1.37 (Pin_37), J1.38 (Pin_38); no longer C31.1
- net GND: no longer names the net of C31.2, C32.2, C33.2, C34.2
- net GND: now also J1.1 (Pin_1), J1.11 (Pin_11), J1.12 (Pin_12), J1.13 (Pin_13), J1.14 (Pin_14), J1.17 (Pin_17), J1.2 (Pin_2), J1.22 (Pin_22), J1.28 (Pin_28), J1.29 (Pin_29), J1.3 (Pin_3), J1.33 (Pin_33), J1.34 (Pin_34), J1.39 (Pin_39), J1.4 (Pin_4), J1.40 (Pin_40)
- net VDD_NVDC renamed VDD_DISP_3V3
- net VDD_DISP_3V3: now also C31.1, J1.10 (Pin_10), J1.5 (Pin_5), J1.6 (Pin_6), J1.7 (Pin_7), J1.8 (Pin_8), J1.9 (Pin_9); no longer C34.1
- new net SPARE_0: J1.16 (Pin_16)
- new net SPARE_1: J1.18 (Pin_18)
- new net SPARE_2: J1.20 (Pin_20)
- new net STATUS_LED_EXT: J1.15 (Pin_15)
Other:
- note removed: "Data"
- note removed: "Power"

Commit message: schematic tidy up, component placement, shielding investigation
Connections:
- net at C31.2, C32.2, C33.2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: no longer J1.13 (Pin_13), J1.14 (Pin_14)
- net VCC_BKUP_3V3 renamed VDD_NVDC
Other:
- moved on the sheet: C31, C32, C33, C34, J1
