File: hardware/mech.kicad_sch (KiCad schematic)
At the start: 7 parts

Commit message: Updates
Parts:
- removed N3: ShieldCan_ESP, RF_Shielding:Laird_Technologies_BMI-S-101_13.66x12.70mm, symbol Mechanical:Housing_Pad
Changed lines of the file:
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@@
-    (stroke (width 0) (type default) (color 0 0 0 0))
-  )
-  (wire (pts (xy 96.52 73.66) (xy 96.52 72.39))
     (stroke (width 0) (type default) (color 0 0 0 0))
   )
@@
     )
   )
-  (symbol (lib_id "power:GND") (at 96.52 73.66 0) (unit 1)
-    (in_bom yes) (on_board yes) (fields_autoplaced)
-    (property "Reference" "#PWR0117" (id 0) (at 96.52 80.01 0)
-      (effects (font (size 0.8 0.8)) hide)
-    )
-    (property "Value" "GND" (id 1) (at 96.52 78.74 0)
-      (effects (font (size 0.8 0.8)) hide)
-    )
-    (property "Footprint" "" (id 2) (at 96.52 73.66 0)
-      (effects (font (size 0.8 0.8)) hide)
-    )
-    (property "Datasheet" "" (id 3) (at 96.52 73.66 0)
-      (effects (font (size 0.8 0.8)) hide)
-    )
-    (pin "1")
-  )
   (symbol (lib_id "Mechanical:Housing") (at 154.94 82.55 0) (unit 1)
     (in_bom yes) (on_board yes)
@@
     )
   )
-  (symbol (lib_id "Mechanical:Housing_Pad") (at 101.6 67.31 0) (unit 1)
-    (in_bom yes) (on_board yes)
-    (property "Reference" "N3" (id 0) (at 106.68 64.77 0)
-      (effects (font (size 1.27 1.27)) (justify left))
-    )
-    (property "Value" "ShieldCan_ESP" (id 1) (at 106.68 67.31 0)
-      (effects (font (size 1.27 1.27)) (justify left))
-    )
-    (property "Footprint" "RF_Shielding:Laird_Technologies_BMI-S-101_13.66x12.70mm" (id 2) (at 103.505 66.04 0)
-      (effects (font (size 1.27 1.27)) hide)
-    )
-    (property "Datasheet" "~" (id 3) (at 103.505 66.04 0)
-      (effects (font (size 1.27 1.27)) hide)
-    )
-    (pin "1")
-  )
   (symbol (lib_id "power:GND") (at 81.28 45.72 0) (unit 1)
