File: hardware/sensors.kicad_sch (KiCad schematic)
At the start: 11 parts, among them U2 FXOS8700CQR1, U3 MS5637-02BA03

Commit message: minor sch tweaks, more layout, added power emc shield
Parts:
- C11: footprint Capacitor_SMD:C_0402_1005Metric -> Capacitor_SMD:C_0603_1608Metric
Connections:
- net GND: now also C15.2, U3.4 (GND)
Changed lines of the file:
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@@
   (junction (at 95.25 123.19) (diameter 0) (color 0 0 0 0)
+  )
+  (junction (at 130.81 85.09) (diameter 0) (color 0 0 0 0)
   )
   (junction (at 121.92 123.19) (diameter 0) (color 0 0 0 0)
@@
     (stroke (width 0) (type default) (color 0 0 0 0))
   )
+  (wire (pts (xy 130.81 86.36) (xy 130.81 85.09))
+    (stroke (width 0) (type default) (color 0 0 0 0))
+  )
   (wire (pts (xy 161.29 77.47) (xy 148.59 77.47))
     (stroke (width 0) (type default) (color 0 0 0 0))
@@
     (pin "1")
   )
+  (symbol (lib_id "power:GND") (at 130.81 86.36 0) (unit 1)
+    (in_bom yes) (on_board yes) (fields_autoplaced)
+    (property "Reference" "#PWR0118" (id 0) (at 130.81 92.71 0)
+      (effects (font (size 1.27 1.27)) hide)
+    )
+    (property "Value" "GND" (id 1) (at 130.81 91.44 0)
+      (effects (font (size 1.27 1.27)) hide)
+    )
+    (property "Footprint" "" (id 2) (at 130.81 86.36 0)
+      (effects (font (size 1.27 1.27)) hide)
+    )
+    (property "Datasheet" "" (id 3) (at 130.81 86.36 0)
+      (effects (font (size 1.27 1.27)) hide)
+    )
+    (pin "1")
+  )
   (symbol (lib_id "Device:C_Small") (at 95.25 113.03 0) (mirror y) (unit 1)
     (in_bom yes) (on_board yes)
@@
       (effects (font (size 0.8 0.8)) (justify left))
     )
-    (property "Footprint" "Capacitor_SMD:C_0402_1005Metric" (id 2) (at 95.25 113.03 0)
-      (effects (font (size 0.8 0.8)) hide)
-    )
+    (property "Footprint" "Capacitor_SMD:C_0603_1608Metric" (id 2) (at 95.25 113.03 0)
+      (effects (font (size 0.8 0.8)) hide)
+    )

Commit message: layout 0 unconnected
Connections:
- net VDD_AUX_3V3 is gone; now on net +3V3: C11.1, C12.1, C15.1, R3.1, R4.1, U2.14 (VDD), U3.1 (VDD)
- net +3V3: now reaches C13.1, U2.1 (VDDIO)
- net SENSOR_I2C.SCL renamed SYS_I2C.SCL
- net SENSOR_I2C.SDA renamed SYS_I2C.SDA
Changed lines of the file:
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@@
     (company "Frisius")
   )
+  (junction (at 110.49 102.87) (diameter 0) (color 0 0 0 0)
+  )
   (junction (at 161.29 68.58) (diameter 0) (color 0 0 0 0)
   )
   (junction (at 95.25 123.19) (diameter 0) (color 0 0 0 0)
+  )
+  (junction (at 118.11 102.87) (diameter 0) (color 0 0 0 0)
   )
   (junction (at 130.81 85.09) (diameter 0) (color 0 0 0 0)
@@
     (stroke (width 0) (type default) (color 0 0 0 0))
   )
+  (wire (pts (xy 118.11 105.41) (xy 118.11 102.87))
+    (stroke (width 0) (type default) (color 0 0 0 0))
+  )
   (wire (pts (xy 149.86 130.81) (xy 149.86 129.54))
     (stroke (width 0) (type default) (color 0 0 0 0))
@@
     (stroke (width 0) (type default) (color 0 0 0 0))
   )
-  (wire (pts (xy 102.87 102.87) (xy 123.19 102.87))
+  (wire (pts (xy 102.87 102.87) (xy 110.49 102.87))
     (stroke (width 0) (type default) (color 0 0 0 0))
   )
@@
     (stroke (width 0) (type default) (color 0 0 0 0))
   )
+  (wire (pts (xy 123.19 105.41) (xy 118.11 105.41))
+    (stroke (width 0) (type default) (color 0 0 0 0))
+  )
   (wire (pts (xy 118.11 115.57) (xy 118.11 123.19))
     (stroke (width 0) (type default) (color 0 0 0 0))
@@
     (stroke (width 0) (type default) (color 0 0 0 0))
   )
-  (wire (pts (xy 110.49 105.41) (xy 110.49 110.49))
+  (wire (pts (xy 110.49 102.87) (xy 110.49 110.49))
     (stroke (width 0) (type default) (color 0 0 0 0))
   )
@@
     (stroke (width 0) (type default) (color 0 0 0 0))
   )
-  (wire (pts (xy 110.49 105.41) (xy 123.19 105.41))
-    (stroke (width 0) (type default) (color 0 0 0 0))
-  )
   (wire (pts (xy 148.59 123.19) (xy 149.86 123.19))
     (stroke (width 0) (type default) (color 0 0 0 0))
@@
     (stroke (width 0) (type default) (color 0 0 0 0))
   )
+  (wire (pts (xy 110.49 102.87) (xy 118.11 102.87))
+    (stroke (width 0) (type default) (color 0 0 0 0))
+  )
   (wire (pts (xy 95.25 74.93) (xy 95.25 77.47))
     (stroke (width 0) (type default) (color 0 0 0 0))
@@
   )
   (wire (pts (xy 95.25 123.19) (xy 102.87 123.19))
+    (stroke (width 0) (type default) (color 0 0 0 0))
+  )
+  (wire (pts (xy 118.11 102.87) (xy 123.19 102.87))
     (stroke (width 0) (type default) (color 0 0 0 0))
   )
@@
     (effects (font (size 1.27 1.27)) (justify left bottom))
   )
-  (label "SENSOR_I2C.SDA" (at 181.61 77.47 0)
+  (label "SYS_I2C.SDA" (at 181.61 77.47 0)
     (effects (font (size 1.27 1.27)) (justify left bottom))
   )
-  (label "SENSOR_I2C.SCL" (at 181.61 80.01 0)
+  (label "SYS_I2C.SCL" (at 181.61 80.01 0)
     (effects (font (size 1.27 1.27)) (justify left bottom))
   )
-  (hierarchical_label "SENSOR_I2C{SDA SCL}" (shape bidirectional) (at 203.2 72.39 0)
+  (hierarchical_label "SYS_I2C{SDA SCL}" (shape bidirectional) (at 203.2 72.39 0)
     (effects (font (size 0.8 0.8)) (justify left))
   )
@@
     (pin "2")
   )
+  (symbol (lib_id "power:+3V3") (at 95.25 74.93 0) (unit 1)
+    (in_bom yes) (on_board yes) (fields_autoplaced)
+    (property "Reference" "#PWR0142" (id 0) (at 95.25 78.74 0)
+      (effects (font (size 1.27 1.27)) hide)
+    )
+    (property "Value" "+3V3" (id 1) (at 95.25 69.85 0))
+    (property "Footprint" "" (id 2) (at 95.25 74.93 0)
+      (effects (font (size 1.27 1.27)) hide)
+    )
+    (property "Datasheet" "" (id 3) (at 95.25 74.93 0)
+      (effects (font (size 1.27 1.27)) hide)
+    )
+    (pin "1")
+  )
+  (symbol (lib_id "power:+3V3") (at 161.29 67.31 0) (unit 1)
+    (in_bom yes) (on_board yes) (fields_autoplaced)
+    (property "Reference" "#PWR0141" (id 0) (at 161.29 71.12 0)
+      (effects (font (size 1.27 1.27)) hide)
+    )
+    (property "Value" "+3V3" (id 1) (at 161.29 62.23 0))
+    (property "Footprint" "" (id 2) (at 161.29 67.31 0)
+      (effects (font (size 1.27 1.27)) hide)
+    )
+    (property "Datasheet" "" (id 3) (at 161.29 67.31 0)
+      (effects (font (size 1.27 1.27)) hide)
+    )
+    (pin "1")
+  )
   (symbol (lib_id "power:GND") (at 121.92 130.81 0) (unit 1)
     (in_bom yes) (on_board yes) (fields_autoplaced)
@@
     )
     (property "Datasheet" "" (id 3) (at 151.13 110.49 0)
-      (effects (font (size 1.27 1.27)) hide)
-    )
-    (pin "1")
-  )
-  (symbol (lib_id "bt_power:VDD_AUX_3V3") (at 95.25 74.93 0) (unit 1)
-    (in_bom no) (on_board no)
-    (property "Reference" "#U02" (id 0) (at 95.7834 74.93 0)
-      (effects (font (size 1.27 1.27)) hide)
-    )
-    (property "Value" "VDD_AUX_3V3" (id 1) (at 95.25 71.12 0))
-    (property "Footprint" "" (id 2) (at 95.7834 74.93 0)
-      (effects (font (size 1.27 1.27)) hide)
-    )
-    (property "Datasheet" "" (id 3) (at 95.7834 74.93 0)
       (effects (font (size 1.27 1.27)) hide)
     )
@@
     (pin "2")
   )
-  (symbol (lib_id "bt_power:VDD_AUX_3V3") (at 161.29 67.31 0) (unit 1)
-    (in_bom no) (on_board no)
-    (property "Reference" "#U03" (id 0) (at 161.8234 67.31 0)
-      (effects (font (size 1.27 1.27)) hide)
-    )
-    (property "Value" "VDD_AUX_3V3" (id 1) (at 161.29 63.5 0))
-    (property "Footprint" "" (id 2) (at 161.8234 67.31 0)
-      (effects (font (size 1.27 1.27)) hide)
-    )
-    (property "Datasheet" "" (id 3) (at 161.8234 67.31 0)
-      (effects (font (size 1.27 1.27)) hide)
-    )
-    (pin "1")
-  )
 )
