File: hardware/base/sdcard.kicad_sch (KiCad schematic)
At the start: 3 parts, among them J1 MEM2067

Commit message: schematic complete unreviewed
Parts:
- removed U?: CM1624, symbol bt_Protection:CM1624
- added C40: 4.7u, Capacitor_SMD:C_0603_1608Metric, symbol Device:C_Small
- added R52, R53, R54: 0, Resistor_SMD:R_0402_1005Metric, symbol Device:R_Small
- added U14: EClamp2410P, bt_Package_DFN:UDFN-16-4x1.6_P0.5mm_EP3x0.5mm, symbol bt_Protection:EClamp2410P
Connections:
- net GND: now also C40.2, U14.17 (GND)
- net SDMMC.CLK: now also U14.3 (CLK_I)
- net SDMMC.CMD: now also U14.6 (CMD_I)
- net SDMMC.D0: now also U14.2 (DAT0_I)
- net SDMMC.D1: now also U14.1 (DAT1_I)
- net SDMMC.D2: now also U14.7 (DAT3_I)
- net SDMMC.D3: now also U14.8 (DAT2_I)
- net at J1.8 (DAT1): now also U14.16 (DAT1_O)
- net at J1.7 (DAT0): now also U14.15 (DAT0_O)
- net at J1.5 (CLK): now also U14.14 (CLK_O)
- net at J1.3 (CMD): now also U14.11 (CMD_O)
- net at J1.2 (DAT3/CD): now also U14.10 (DAT3_O)
- net at J1.1 (DAT2): now also U14.9 (DAT2_O)
- net +3V3 renamed VDD_AUX_3V3
- net VDD_AUX_3V3: now also C40.1, R52.2, R53.2, R54.2, U14.5 (VDD)
- new net: R52.1, U14.4 (Rup1)
- new net: R53.1, U14.12 (Rup2)
- new net: R54.1, U14.13 (Rup3)
Other:
- moved on the sheet: C3

Commit message: placed components on board - rough
Parts:
- removed C40: 4.7u, Capacitor_SMD:C_0603_1608Metric, symbol Device:C_Small
Changed lines of the file:
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@@
   (junction (at 113.03 74.93) (diameter 0) (color 0 0 0 0)
   )
-  (junction (at 104.14 74.93) (diameter 0) (color 0 0 0 0)
-  )
   (junction (at 100.33 74.93) (diameter 0) (color 0 0 0 0)
   )
@@
     (stroke (width 0) (type default) (color 0 0 0 0))
   )
-  (wire (pts (xy 100.33 74.93) (xy 104.14 74.93))
-    (stroke (width 0) (type default) (color 0 0 0 0))
-  )
   (wire (pts (xy 115.57 83.82) (xy 113.03 83.82))
     (stroke (width 0) (type default) (color 0 0 0 0))
@@
     (stroke (width 0) (type default) (color 0 0 0 0))
   )
-  (wire (pts (xy 104.14 81.28) (xy 104.14 83.185))
-    (stroke (width 0) (type default) (color 0 0 0 0))
-  )
   (wire (pts (xy 154.305 91.44) (xy 152.4 91.44))
     (stroke (width 0) (type default) (color 0 0 0 0))
@@
     (stroke (width 0) (type default) (color 0 0 0 0))
   )
-  (wire (pts (xy 104.14 74.93) (xy 113.03 74.93))
+  (wire (pts (xy 100.33 74.93) (xy 113.03 74.93))
     (stroke (width 0) (type default) (color 0 0 0 0))
   )
@@
   )
   (wire (pts (xy 113.03 88.9) (xy 113.03 86.36))
-    (stroke (width 0) (type default) (color 0 0 0 0))
-  )
-  (wire (pts (xy 104.14 76.2) (xy 104.14 74.93))
     (stroke (width 0) (type default) (color 0 0 0 0))
   )
@@
     (property "Datasheet" "~" (id 3) (at 118.11 83.82 0)
       (effects (font (size 0.8 0.8)) hide)
-    )
-    (pin "1")
-    (pin "2")
-  )
-  (symbol (lib_id "Device:C_Small") (at 104.14 78.74 0) (unit 1)
-    (in_bom yes) (on_board yes)
-    (property "Reference" "C40" (id 0) (at 106.68 77.47 0)
-      (effects (font (size 0.8 0.8)) (justify left))
-    )
-    (property "Value" "4.7u" (id 1) (at 106.68 78.74 0)
-      (effects (font (size 0.8 0.8)) (justify left))
-    )
-    (property "Footprint" "Capacitor_SMD:C_0603_1608Metric" (id 2) (at 104.14 78.74 0)
-      (effects (font (size 0.8 0.8)) hide)
-    )
-    (property "Datasheet" "~" (id 3) (at 104.14 78.74 0)
-      (effects (font (size 0.8 0.8)) hide)
-    )
-    (property "Voltage" "15V" (id 4) (at 106.68 80.01 0)
-      (effects (font (size 0.8 0.8)) (justify left))
     )
     (pin "1")
@@
     (pin "9")
   )
-  (symbol (lib_id "power:GND") (at 104.14 83.185 0) (unit 1)
-    (in_bom yes) (on_board yes)
-    (property "Reference" "#PWR0145" (id 0) (at 104.14 89.535 0)
-      (effects (font (size 0.8 0.8)) hide)
-    )
-    (property "Value" "GND" (id 1) (at 104.14 86.995 0)
-      (effects (font (size 0.8 0.8)) hide)
-    )
-    (property "Footprint" "" (id 2) (at 104.14 83.185 0)
-      (effects (font (size 0.8 0.8)) hide)
-    )
-    (property "Datasheet" "" (id 3) (at 104.14 83.185 0)
-      (effects (font (size 0.8 0.8)) hide)
-    )
-    (pin "1")
-  )
   (symbol (lib_id "bt_power:VDD_AUX_3V3") (at 100.33 72.39 0) (unit 1)

Commit message: layout
Connections:
- net cl_r1: now reaches R52.1, U14.4 (Rup1)
- net sd_d2: now reaches J1.1 (DAT2), U14.9 (DAT2_O)
- net sd_d3: now reaches J1.2 (DAT3/CD), U14.10 (DAT3_O)
- net sd_cmd: now reaches J1.3 (CMD), U14.11 (CMD_O)
- net sd_clk: now reaches J1.5 (CLK), U14.14 (CLK_O)
- net sd_d0: now reaches J1.7 (DAT0), U14.15 (DAT0_O)
- net sd_d1: now reaches J1.8 (DAT1), U14.16 (DAT1_O)
- net cl_r2: now reaches R53.1, U14.12 (Rup2)
- net cl_r3: now reaches R54.1, U14.13 (Rup3)
Changed lines of the file:
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@@
     (stroke (width 0) (type default) (color 0 0 0 0))
   )
+  (label "sd_d1" (at 144.78 101.6 0)
+    (effects (font (size 0.8 0.8)) (justify left bottom))
+  )
   (label "SDMMC.CMD" (at 113.03 95.25 0)
+    (effects (font (size 0.8 0.8)) (justify left bottom))
+  )
+  (label "sd_cmd" (at 144.78 88.9 0)
+    (effects (font (size 0.8 0.8)) (justify left bottom))
+  )
+  (label "cl_r2" (at 121.92 86.36 0)
+    (effects (font (size 0.8 0.8)) (justify left bottom))
+  )
+  (label "sd_d3" (at 144.78 86.36 0)
+    (effects (font (size 0.8 0.8)) (justify left bottom))
+  )
+  (label "sd_clk" (at 144.78 93.98 0)
+    (effects (font (size 0.8 0.8)) (justify left bottom))
+  )
+  (label "sd_d0" (at 144.78 99.06 0)
     (effects (font (size 0.8 0.8)) (justify left bottom))
   )
@@
     (effects (font (size 0.8 0.8)) (justify left bottom))
   )
+  (label "sd_d2" (at 144.78 83.82 0)
+    (effects (font (size 0.8 0.8)) (justify left bottom))
+  )
   (label "SDMMC.D0" (at 113.03 97.79 0)
     (effects (font (size 0.8 0.8)) (justify left bottom))
   )
+  (label "cl_r3" (at 121.92 88.9 0)
+    (effects (font (size 0.8 0.8)) (justify left bottom))
+  )
+  (label "cl_r1" (at 121.92 83.82 0)
+    (effects (font (size 0.8 0.8)) (justify left bottom))
+  )
