File: hardware/base/usb.kicad_sch (KiCad schematic)
At the start: 69 parts, among them J2 USB_C_Receptacle_USB2.0, J3 BATTERY, J7 I2C ISENSE, Q2 Q_NMOS_DGS, Q3 Q_NMOS_DGS, SW3 POWER, U12 PAC1944, U13 TLV62569DBV/AP3428, U7 TLV62569DBV/AP3428, U8 MP2723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

Commit message: placed components on board - rough
Connections:
- net VAUX_S+: now also U12.8 (IN3+); no longer U12.10 (IN4+)
- net VAUX_S-: now also U12.7 (IN3-); no longer U12.9 (IN4-)
- net VCORE_S+: now also U12.10 (IN4+); no longer U12.8 (IN3+)
- net VCORE_S-: now also U12.9 (IN4-); no longer U12.7 (IN3-)
- net EP renamed GND

Commit message: further placement, pre condense
Connections:
- net ISENSE_SCL: now also J7.3 (Pin_3); no longer J7.2 (Pin_2)
- net ISENSE_SDA: now also J7.2 (Pin_2); no longer J7.3 (Pin_3)
Changed lines of the file:
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@@
   (junction (at 49.53 66.04) (diameter 0) (color 0 0 0 0)
   )
+  (junction (at 161.29 129.54) (diameter 0) (color 0 0 0 0)
+  )
   (junction (at 227.33 139.7) (diameter 0) (color 0 0 0 0)
-  )
-  (junction (at 161.29 129.54) (diameter 0) (color 0 0 0 0)
   )
   (junction (at 31.75 152.4) (diameter 0) (color 0 0 0 0)
@@
     (stroke (width 0) (type default) (color 0 0 0 0))
   )
+  (wire (pts (xy 227.33 139.7) (xy 232.41 139.7))
+    (stroke (width 0) (type default) (color 0 0 0 0))
+  )
   (wire (pts (xy 179.07 36.83) (xy 168.91 36.83))
     (stroke (width 0) (type default) (color 0 0 0 0))
@@
     (stroke (width 0) (type default) (color 0 0 0 0))
   )
-  (wire (pts (xy 231.14 151.13) (xy 224.79 151.13))
-    (stroke (width 0) (type default) (color 0 0 0 0))
-  )
   (wire (pts (xy 31.75 146.05) (xy 31.75 152.4))
     (stroke (width 0) (type default) (color 0 0 0 0))
@@
     (stroke (width 0) (type default) (color 0 0 0 0))
   )
+  (wire (pts (xy 231.14 148.59) (xy 224.79 148.59))
+    (stroke (width 0) (type default) (color 0 0 0 0))
+  )
   (wire (pts (xy 88.9 158.75) (xy 88.9 167.64))
     (stroke (width 0) (type default) (color 0 0 0 0))
@@
     (stroke (width 0) (type default) (color 0 0 0 0))
   )
+  (wire (pts (xy 231.14 151.13) (xy 227.33 151.13))
+    (stroke (width 0) (type default) (color 0 0 0 0))
+  )
   (wire (pts (xy 137.16 175.26) (xy 130.81 175.26))
     (stroke (width 0) (type default) (color 0 0 0 0))
@@
     (stroke (width 0) (type default) (color 0 0 0 0))
   )
-  (wire (pts (xy 231.14 148.59) (xy 227.33 148.59))
-    (stroke (width 0) (type default) (color 0 0 0 0))
-  )
   (wire (pts (xy 138.43 58.42) (xy 143.51 58.42))
     (stroke (width 0) (type default) (color 0 0 0 0))
@@
     (stroke (width 0) (type default) (color 0 0 0 0))
   )
-  (wire (pts (xy 224.79 142.24) (xy 224.79 151.13))
+  (wire (pts (xy 224.79 142.24) (xy 224.79 148.59))
     (stroke (width 0) (type default) (color 0 0 0 0))
   )
@@
     (stroke (width 0) (type default) (color 0 0 0 0))
   )
-  (wire (pts (xy 227.33 139.7) (xy 232.41 139.7))
-    (stroke (width 0) (type default) (color 0 0 0 0))
-  )
   (wire (pts (xy 213.36 147.32) (xy 215.9 147.32))
     (stroke (width 0) (type default) (color 0 0 0 0))
@@
     (stroke (width 0) (type default) (color 0 0 0 0))
   )
+  (wire (pts (xy 227.33 151.13) (xy 227.33 139.7))
+    (stroke (width 0) (type default) (color 0 0 0 0))
+  )
   (wire (pts (xy 143.51 124.46) (xy 143.51 125.73))
     (stroke (width 0) (type default) (color 0 0 0 0))
@@
     (stroke (width 0) (type default) (color 0 0 0 0))
   )
-  (wire (pts (xy 227.33 139.7) (xy 227.33 148.59))
-    (stroke (width 0) (type default) (color 0 0 0 0))
-  )

Commit message: Testing condensed layout
Parts:
- J7: footprint Connector_PinHeader_2.54mm:PinHeader_1x04_P2.54mm_Vertical -> Connector_PinHeader_1.27mm:PinHeader_1x04_P1.27mm_Vertical
Connections:
- net ISENSE_SCL: now also J7.2 (Pin_2); no longer J7.3 (Pin_3)
- net ISENSE_SDA: now also J7.3 (Pin_3); no longer J7.2 (Pin_2)
Changed lines of the file:
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@@
   (junction (at 153.67 129.54) (diameter 0) (color 0 0 0 0)
   )
+  (junction (at 86.36 48.26) (diameter 0) (color 0 0 0 0)
+  )
+  (junction (at 142.24 68.58) (diameter 0) (color 0 0 0 0)
+  )
+  (junction (at 196.85 60.96) (diameter 0) (color 0 0 0 0)
+  )
+  (junction (at 171.45 55.88) (diameter 0) (color 0 0 0 0)
+  )
+  (junction (at 74.93 158.75) (diameter 0) (color 0 0 0 0)
+  )
+  (junction (at 49.53 63.5) (diameter 0) (color 0 0 0 0)
+  )
+  (junction (at 92.71 167.64) (diameter 0) (color 0 0 0 0)
+  )
+  (junction (at 167.64 88.9) (diameter 0) (color 0 0 0 0)
+  )
+  (junction (at 172.72 99.06) (diameter 0) (color 0 0 0 0)
+  )
+  (junction (at 58.42 71.12) (diameter 0) (color 0 0 0 0)
+  )
+  (junction (at 223.52 68.58) (diameter 0) (color 0 0 0 0)
+  )
+  (junction (at 186.69 33.02) (diameter 0) (color 0 0 0 0)
+  )
+  (junction (at 74.93 48.26) (diameter 0) (color 0 0 0 0)
+  )
+  (junction (at 137.16 167.64) (diameter 0) (color 0 0 0 0)
+  )
+  (junction (at 67.31 48.26) (diameter 0) (color 0 0 0 0)
+  )
+  (junction (at 121.92 48.26) (diameter 0) (color 0 0 0 0)
+  )
+  (junction (at 137.16 129.54) (diameter 0) (color 0 0 0 0)
+  )
+  (junction (at 88.9 142.24) (diameter 0) (color 0 0 0 0)
+  )
   (junction (at 224.79 142.24) (diameter 0) (color 0 0 0 0)
   )
-  (junction (at 86.36 48.26) (diameter 0) (color 0 0 0 0)
-  )
-  (junction (at 142.24 68.58) (diameter 0) (color 0 0 0 0)
-  )
-  (junction (at 196.85 60.96) (diameter 0) (color 0 0 0 0)
-  )
-  (junction (at 171.45 55.88) (diameter 0) (color 0 0 0 0)
-  )
-  (junction (at 74.93 158.75) (diameter 0) (color 0 0 0 0)
-  )
-  (junction (at 49.53 63.5) (diameter 0) (color 0 0 0 0)
-  )
-  (junction (at 92.71 167.64) (diameter 0) (color 0 0 0 0)
-  )
-  (junction (at 167.64 88.9) (diameter 0) (color 0 0 0 0)
-  )
-  (junction (at 172.72 99.06) (diameter 0) (color 0 0 0 0)
-  )
-  (junction (at 58.42 71.12) (diameter 0) (color 0 0 0 0)
-  )
-  (junction (at 223.52 68.58) (diameter 0) (color 0 0 0 0)
-  )
-  (junction (at 186.69 33.02) (diameter 0) (color 0 0 0 0)
-  )
-  (junction (at 74.93 48.26) (diameter 0) (color 0 0 0 0)
-  )
-  (junction (at 137.16 167.64) (diameter 0) (color 0 0 0 0)
-  )
-  (junction (at 67.31 48.26) (diameter 0) (color 0 0 0 0)
-  )
-  (junction (at 121.92 48.26) (diameter 0) (color 0 0 0 0)
-  )
-  (junction (at 137.16 129.54) (diameter 0) (color 0 0 0 0)
-  )
-  (junction (at 88.9 142.24) (diameter 0) (color 0 0 0 0)
-  )
   (junction (at 161.29 167.64) (diameter 0) (color 0 0 0 0)
   )
@@
   (junction (at 215.9 149.86) (diameter 0) (color 0 0 0 0)
   )
+  (junction (at 227.33 139.7) (diameter 0) (color 0 0 0 0)
+  )
   (junction (at 130.81 137.16) (diameter 0) (color 0 0 0 0)
   )
@@
   )
   (junction (at 161.29 129.54) (diameter 0) (color 0 0 0 0)
-  )
-  (junction (at 227.33 139.7) (diameter 0) (color 0 0 0 0)
   )
   (junction (at 31.75 152.4) (diameter 0) (color 0 0 0 0)
@@
     (stroke (width 0) (type default) (color 0 0 0 0))
   )
-  (wire (pts (xy 227.33 139.7) (xy 232.41 139.7))
+  (wire (pts (xy 213.36 139.7) (xy 227.33 139.7))
     (stroke (width 0) (type default) (color 0 0 0 0))
   )
@@
     (stroke (width 0) (type default) (color 0 0 0 0))
   )
+  (wire (pts (xy 224.79 142.24) (xy 232.41 142.24))
+    (stroke (width 0) (type default) (color 0 0 0 0))
+  )
   (wire (pts (xy 137.16 129.54) (xy 137.16 130.81))
     (stroke (width 0) (type default) (color 0 0 0 0))
@@
     (stroke (width 0) (type default) (color 0 0 0 0))
   )
-  (wire (pts (xy 231.14 148.59) (xy 224.79 148.59))
+  (wire (pts (xy 231.14 148.59) (xy 227.33 148.59))
     (stroke (width 0) (type default) (color 0 0 0 0))
   )
@@
   )
   (wire (pts (xy 121.92 132.08) (xy 121.92 137.16))
+    (stroke (width 0) (type default) (color 0 0 0 0))
+  )
+  (wire (pts (xy 227.33 139.7) (xy 232.41 139.7))
     (stroke (width 0) (type default) (color 0 0 0 0))
   )
@@
     (stroke (width 0) (type default) (color 0 0 0 0))
   )
-  (wire (pts (xy 231.14 151.13) (xy 227.33 151.13))
+  (wire (pts (xy 224.79 151.13) (xy 231.14 151.13))
     (stroke (width 0) (type default) (color 0 0 0 0))
   )
@@
     (stroke (width 0) (type default) (color 0 0 0 0))
   )
-  (wire (pts (xy 224.79 142.24) (xy 232.41 142.24))
+  (wire (pts (xy 224.79 151.13) (xy 224.79 142.24))
+    (stroke (width 0) (type default) (color 0 0 0 0))
+  )
+  (wire (pts (xy 213.36 142.24) (xy 224.79 142.24))
     (stroke (width 0) (type default) (color 0 0 0 0))
   )
@@
     (stroke (width 0) (type default) (color 0 0 0 0))
   )
-  (wire (pts (xy 213.36 142.24) (xy 224.79 142.24))
-    (stroke (width 0) (type default) (color 0 0 0 0))
-  )
   (wire (pts (xy 130.81 129.54) (xy 130.81 130.81))
     (stroke (width 0) (type default) (color 0 0 0 0))
@@
     (stroke (width 0) (type default) (color 0 0 0 0))
   )
-  (wire (pts (xy 224.79 142.24) (xy 224.79 148.59))
-    (stroke (width 0) (type default) (color 0 0 0 0))
-  )
   (wire (pts (xy 215.9 147.32) (xy 215.9 149.86))
-    (stroke (width 0) (type default) (color 0 0 0 0))
-  )
-  (wire (pts (xy 213.36 139.7) (xy 227.33 139.7))
     (stroke (width 0) (type default) (color 0 0 0 0))
   )
@@
     (stroke (width 0) (type default) (color 0 0 0 0))
   )
-  (wire (pts (xy 227.33 151.13) (xy 227.33 139.7))
-    (stroke (width 0) (type default) (color 0 0 0 0))
-  )
   (wire (pts (xy 143.51 124.46) (xy 143.51 125.73))
     (stroke (width 0) (type default) (color 0 0 0 0))
@@
   )
   (wire (pts (xy 66.04 139.7) (xy 66.04 140.97))
+    (stroke (width 0) (type default) (color 0 0 0 0))
+  )
+  (wire (pts (xy 227.33 148.59) (xy 227.33 139.7))
     (stroke (width 0) (type default) (color 0 0 0 0))
   )
@@
       (effects (font (size 0.8 0.8)))
     )
-    (property "Footprint" "Connector_PinHeader_2.54mm:PinHeader_1x04_P2.54mm_Vertical" (id 2) (at 236.22 151.13 0)
-      (effects (font (size 1.27 1.27)) hide)
-    )
+    (property "Footprint" "Connector_PinHeader_1.27mm:PinHeader_1x04_P1.27mm_Vertical" (id 2) (at 236.22 151.13 0)
+      (effects (font (size 1.27 1.27)) hide)
+    )

Commit message: layout
Connections:
- net VAUX_S+: now also U12.13 (IN2+); no longer U12.8 (IN3+)
- net VAUX_S-: now also U12.14 (IN2-); no longer U12.7 (IN3-)
- net VBAT_S+: now also U12.9 (IN4-); no longer U12.14 (IN2-)
- net VBAT_S-: now also U12.10 (IN4+); no longer U12.13 (IN2+)
- net VBUS_S+: now also U12.8 (IN3+); no longer U12.11 (IN1+)
- net VBUS_S-: now also U12.7 (IN3-); no longer U12.12 (IN1-)
- net VCORE_S+: now also U12.11 (IN1+); no longer U12.10 (IN4+)
- net VCORE_S-: now also U12.12 (IN1-); no longer U12.9 (IN4-)
- net chg_otg: now reaches R44.1, U8.23 (OTG)
- net vaux_fb: now reaches C31.2, R35.2, R43.1, U13.5 (FB)
- net chg_batt: now reaches R50.1, U8.17 (BATT)
- net chg_ilim: now reaches R34.1, U8.24 (ILIM)
- net vcore_fb: now reaches C6.2, R29.2, R30.1, U7.5 (FB)
- net usb_cc2: now reaches J2.B5 (CC2), R22.1
- net chg_ntc: now reaches R36.1, R37.2, U8.11 (NTC)
- net chg_vntc: now reaches R36.2, U8.12 (VNTC)
- net usb_cc1: now reaches J2.A5 (CC1), R21.1
- net bat_ntc: now reaches J3.2 (Pin_2), R37.1
- net chg_vref: now reaches C37.1, R31.1, R32.1, U8.13-14 (VREF)
- net chg_stat_led: now reaches D3.2 (A), R32.2
- net chg_ce: now reaches R46.1, U8.18 (~{CE})
- net chg_disc: now reaches R31.2, U8.22 (DISC)
- net chg_pmid: now reaches C23.1, U8.3 (PMID)
- net chg_sw: now reaches C10.2, L2.1, U8.4 (SW)
- net chg_bst: now reaches C10.1, U8.8 (BST)
- net chg_stat: now reaches D3.1 (K), U8.9 (STAT)
- net PORT_D+ renamed USB_D+
- net PORT_D- renamed USB_D-
Other:
- moved on the sheet: R36, R37

Commit message: more layout, optimising i2c
Parts:
- removed C22: 4.7u, Capacitor_SMD:C_0603_1608Metric, symbol Device:C_Small
Connections:
- net USB_D+: now also D4.2 (K); no longer D4.1 (K)
- net USB_D-: now also D4.1 (K); no longer D4.2 (K)
- net VAUX_S+: now also U12.8 (IN3+); no longer R51.2, U12.13 (IN2+)
- net VAUX_S-: now also U12.7 (IN3-); no longer U12.14 (IN2-)
- net VBAT_S+: now also U12.12 (IN1-); no longer U12.9 (IN4-)
- net VBAT_S-: now also U12.11 (IN1+); no longer U12.10 (IN4+)
- net VBUS_S+: now also U12.9 (IN4-); no longer U12.8 (IN3+)
- net VBUS_S-: now also U12.10 (IN4+); no longer U12.7 (IN3-)
- net VCORE_S+: now also U12.13 (IN2+); no longer U12.11 (IN1+)
- net VCORE_S-: now also U12.14 (IN2-); no longer U12.12 (IN1-)
- net VDD_AUX_3V3: no longer C32.1, C33.1
- net VDD_CORE_3V3: no longer C7.1, C8.1
- net core_drv: now reaches L1.1, U7.3 (SW)
- net vcore_sw: now reaches C6.1, L1.2, R29.1, R45.1
- net vcore_sw: now also C7.1, C8.1
- net vbus_port: now reaches C35.1, C36.1, J2.A4 (VBUS), J2.A9 (VBUS), J2.B4 (VBUS), J2.B9 (VBUS), R42.1
- net aux_sw: now reaches C31.1, L3.2, R35.1, R51.1
- net aux_sw: now also C32.1, C33.1
- net aux_drv: now reaches L3.1, U13.3 (SW)
- net btn_nvdc: now reaches R19.1, SW3.1
Other:
- moved on the sheet: C32, C33, C7, C8, R45, R51

Commit message: layout complete, drc checks and tweaks to silkscreen, attempting geo reannotate
Connections:
- net ISENSE_INT: no longer R47.2
- net VAUX_S+: now also R51.2
- new net SYS_ISENSE_INT: R47.2
Changed lines of the file:
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@@
+    (stroke (width 0) (type default) (color 0 0 0 0))
+  )
+  (wire (pts (xy 154.94 162.56) (xy 154.94 163.83))
     (stroke (width 0) (type default) (color 0 0 0 0))
   )
@@
     (effects (font (size 0.8 0.8)) (justify right))
   )
-  (hierarchical_label "ISENSE_INT" (shape output) (at 238.76 134.62 0)
+  (hierarchical_label "SYS_ISENSE_INT" (shape output) (at 238.76 134.62 0)
     (effects (font (size 0.8 0.8)) (justify left))
   )
