File: hardware/base/processor.kicad_sch (KiCad schematic)
At the start: 20 parts, among them J4 Debug UART, SW1 RESET, SW2 BOOT, SW4 NAV, U1 PI4IOE5V9554A, U10 TCA9801, U3 ESP32-S3-WROOM-1-PinOrder

Commit message: Tidied up, added more stitches
Parts:
- U10: value TCA9801 -> TCA9803
Connections:
- net GND: now also U10.4 (GND)
Changed lines of the file:
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@@
+    (stroke (width 0) (type default) (color 0 0 0 0))
+  )
+  (wire (pts (xy 242.57 146.05) (xy 242.57 145.415))
     (stroke (width 0) (type default) (color 0 0 0 0))
   )
@@
     (pin "2")
   )
+  (symbol (lib_id "power:GND") (at 242.57 146.05 0) (mirror y) (unit 1)
+    (in_bom yes) (on_board yes)
+    (property "Reference" "#PWR0164" (id 0) (at 242.57 152.4 0)
+      (effects (font (size 1.27 1.27)) hide)
+    )
+    (property "Value" "GND" (id 1) (at 242.57 151.13 0))
+    (property "Footprint" "" (id 2) (at 242.57 146.05 0)
+      (effects (font (size 1.27 1.27)) hide)
+    )
+    (property "Datasheet" "" (id 3) (at 242.57 146.05 0)
+      (effects (font (size 1.27 1.27)) hide)
+    )
+    (pin "1")
+  )
   (symbol (lib_id "Device:R_Small") (at 39.37 45.72 0) (mirror y) (unit 1)
     (in_bom yes) (on_board yes)
@@
   (symbol (lib_id "Interface:TCA9801") (at 242.57 132.715 0) (unit 1)
     (in_bom yes) (on_board yes) (fields_autoplaced)
-    (property "Reference" "U10" (id 0) (at 244.5894 145.415 0)
-      (effects (font (size 1.27 1.27)) (justify left))
-    )
-    (property "Value" "TCA9801" (id 1) (at 244.5894 147.955 0)
-      (effects (font (size 1.27 1.27)) (justify left))
-    )
+    (property "Reference" "U10" (id 0) (at 244.5894 146.05 0)
+      (effects (font (size 1.27 1.27)) (justify left))
+    )
+    (property "Value" "TCA9803" (id 1) (at 244.5894 148.59 0)
+      (effects (font (size 1.27 1.27)) (justify left))
+    )
